Commit message: change urdf path

File: src/hexapod_description/robot/visual/hexapod.urdf (robot description, URDF)
Before this commit: robot URDF_Full_Hexapod, 31 links, 30 joints
Links:
- link ankle_link_1: geometry collision mesh filename=/home/ambushee/FRA333_Kinematic_Project/src/hexapod_descrip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; visual mesh filename=/home/ambushee/FRA333_Kinematic_Project/src/hexapod_descrip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
- link ankle_link_2: geometry collision mesh filename=/home/ambushee/FRA333_Kinematic_Project/src/hexapod_descrip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; visual mesh filename=/home/ambushee/FRA333_Kinematic_Project/src/hexapod_descrip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
- link ankle_link_3: geometry collision mesh filename=/home/ambushee/FRA333_Kinematic_Project/src/hexapod_descrip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; visual mesh filename=/home/ambushee/FRA333_Kinematic_Project/src/hexapod_descrip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
- link ankle_link_4: geometry collision mesh filename=/home/ambushee/FRA333_Kinematic_Project/src/hexapod_descrip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; visual mesh filename=/home/ambushee/FRA333_Kinematic_Project/src/hexapod_descrip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
- link ankle_link_5: geometry collision mesh filename=/home/ambushee/FRA333_Kinematic_Project/src/hexapod_descrip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; visual mesh filename=/home/ambushee/FRA333_Kinematic_Project/src/hexapod_descrip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
- link ankle_link_6: geometry collision mesh filename=/home/ambushee/FRA333_Kinematic_Project/src/hexapod_descrip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; visual mesh filename=/home/ambushee/FRA333_Kinematic_Project/src/hexapod_descrip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
- link base_link: geometry collision mesh filename=/home/ambushee/FRA333_Kinematic_Project/src/hexapod_descrip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; visual mesh filename=/home/ambushee/FRA333_Kinematic_Project/src/hexapod_descrip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
- link end_effector_1: geometry collision mesh filename=/home/ambushee/FRA333_Kinematic_Project/src/hexapod_descrip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; visual mesh filename=/home/ambushee/FRA333_Kinematic_Project/src/hexapod_descrip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
- link end_effector_2: geometry collision mesh filename=/home/ambushee/FRA333_Kinematic_Project/src/hexapod_descrip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; visual mesh filename=/home/ambushee/FRA333_Kinematic_Project/src/hexapod_descrip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
- link end_effector_3: geometry collision mesh filename=/home/ambushee/FRA333_Kinematic_Project/src/hexapod_descrip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; visual mesh filename=/home/ambushee/FRA333_Kinematic_Project/src/hexapod_descrip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
- link end_effector_4: geometry collision mesh filename=/home/ambushee/FRA333_Kinematic_Project/src/hexapod_descrip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; visual mesh filename=/home/ambushee/FRA333_Kinematic_Project/src/hexapod_descrip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
- link end_effector_5: geometry collision mesh filename=/home/ambushee/FRA333_Kinematic_Project/src/hexapod_descrip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; visual mesh filename=/home/ambushee/FRA333_Kinematic_Project/src/hexapod_descrip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
- link end_effector_6: geometry collision mesh filename=/home/ambushee/FRA333_Kinematic_Project/src/hexapod_descrip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; visual mesh filename=/home/ambushee/FRA333_Kinematic_Project/src/hexapod_descrip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
- link foot_pointer_1: geometry collision mesh filename=/home/ambushee/FRA333_Kinematic_Project/src/hexapod_descrip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; visual mesh filename=/home/ambushee/FRA333_Kinematic_Project/src/hexapod_descrip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
- link foot_pointer_2: geometry collision mesh filename=/home/ambushee/FRA333_Kinematic_Project/src/hexapod_descrip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; visual mesh filename=/home/ambushee/FRA333_Kinematic_Project/src/hexapod_descrip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
- link foot_pointer_3: geometry collision mesh filename=/home/ambushee/FRA333_Kinematic_Project/src/hexapod_descrip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; visual mesh filename=/home/ambushee/FRA333_Kinematic_Project/src/hexapod_descrip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
- link foot_pointer_4: geometry collision mesh filename=/home/ambushee/FRA333_Kinematic_Project/src/hexapod_descrip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; visual mesh filename=/home/ambushee/FRA333_Kinematic_Project/src/hexapod_descrip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
- link foot_pointer_5: geometry collision mesh filename=/home/ambushee/FRA333_Kinematic_Project/src/hexapod_descrip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; visual mesh filename=/home/ambushee/FRA333_Kinematic_Project/src/hexapod_descrip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
- link foot_pointer_6: geometry collision mesh filename=/home/ambushee/FRA333_Kinematic_Project/src/hexapod_descrip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; visual mesh filename=/home/ambushee/FRA333_Kinematic_Project/src/hexapod_descrip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
- link hip_link_1: geometry collision mesh filename=/home/ambushee/FRA333_Kinematic_Project/src/hexapod_descrip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; visual mesh filename=/home/ambushee/FRA333_Kinematic_Project/src/hexapod_descrip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
- link hip_link_2: geometry collision mesh filename=/home/ambushee/FRA333_Kinematic_Project/src/hexapod_descrip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; visual mesh filename=/home/ambushee/FRA333_Kinematic_Project/src/hexapod_descrip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
- link hip_link_3: geometry collision mesh filename=/home/ambushee/FRA333_Kinematic_Project/src/hexapod_descrip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; visual mesh filename=/home/ambushee/FRA333_Kinematic_Project/src/hexapod_descrip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
- link hip_link_4: geometry collision mesh filename=/home/ambushee/FRA333_Kinematic_Project/src/hexapod_descrip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; visual mesh filename=/home/ambushee/FRA333_Kinematic_Project/src/hexapod_descrip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
- link hip_link_5: geometry collision mesh filename=/home/ambushee/FRA333_Kinematic_Project/src/hexapod_descrip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; visual mesh filename=/home/ambushee/FRA333_Kinematic_Project/src/hexapod_descrip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
- link hip_link_6: geometry collision mesh filename=/home/ambushee/FRA333_Kinematic_Project/src/hexapod_descrip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; visual mesh filename=/home/ambushee/FRA333_Kinematic_Project/src/hexapod_descrip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
- link knee_link_1: geometry collision mesh filename=/home/ambushee/FRA333_Kinematic_Project/src/hexapod_descrip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; visual mesh filename=/home/ambushee/FRA333_Kinematic_Project/src/hexapod_descrip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
- link knee_link_2: geometry collision mesh filename=/home/ambushee/FRA333_Kinematic_Project/src/hexapod_descrip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; visual mesh filename=/home/ambushee/FRA333_Kinematic_Project/src/hexapod_descrip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
- link knee_link_3: geometry collision mesh filename=/home/ambushee/FRA333_Kinematic_Project/src/hexapod_descrip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; visual mesh filename=/home/ambushee/FRA333_Kinematic_Project/src/hexapod_descrip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
- link knee_link_4: geometry collision mesh filename=/home/ambushee/FRA333_Kinematic_Project/src/hexapod_descrip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; visual mesh filename=/home/ambushee/FRA333_Kinematic_Project/src/hexapod_descrip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
- link knee_link_5: geometry collision mesh filename=/home/ambushee/FRA333_Kinematic_Project/src/hexapod_descrip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; visual mesh filename=/home/ambushee/FRA333_Kinematic_Project/src/hexapod_descrip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
- link knee_link_6: geometry collision mesh filename=/home/ambushee/FRA333_Kinematic_Project/src/hexapod_descrip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; visual mesh filename=/home/ambushee/FRA333_Kinematic_Project/src/hexapod_descrip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
