Commit message: Add Joint Trajectory Controller implementation for hexapod simulation
Major Changes:
- Implemented trajectory controller bridge for converting IK output to JointTrajectory messages
- Created new URDF configuration (hexapod_trajectory.xacro) with position command interface
- Added Gazebo configuration for trajectory controllers (gazebo_trajectory.xacro)
- Implemented gravity compensation node for improved control accuracy
- Created new launch file for trajectory controller simulation

New Files:
- src/hexapod/scripts/trajectory_controller_bridge.py: Bridge between IK and trajectory controllers
- src/hexapod/scripts/gravity_compensation.py: Gravity compensation implementation
- src/hexapod_description/robot/visual/hexapod_trajectory.xacro: URDF with corrected hip positions
- src/hexapod_description/robot/visual/gazebo_trajectory.xacro: Gazebo config with position control
- src/hexapod_simulation/config/controller_trajectory.yaml: Trajectory controller configuration
- src/hexapod_simulation/launch/simulation-trajectory.launch.py: Launch file for trajectory control

Fixes:
- Fixed mesh rendering issue in Gazebo by adding Sensors plugin
- Corrected hip joint positions from rectangular to hexagonal layout
- Fixed environment variable setup for Gazebo resource paths
- Updated controller interface from effort to position command

Testing Results:
- ✅ Mesh rendering works correctly in Gazebo
- ✅ Hip positions are accurate (hexagonal layout)
- ✅ Trajectory controllers accept and execute commands
- ✅ Joints move according to trajectory setpoints

🤖 Generated with Claude Code
Co-Authored-By: Claude <noreply@anthropic.com>

File: src/hexapod_description/robot/visual/hexapod.urdf (robot description, URDF)
Before this commit: robot URDF_Full_Hexapod, 31 links, 30 joints
Links:
- added link foot_contact_1, mass 0.001; collision sphere radius=0.01; visual sphere radius=0.01
- added link foot_contact_2, mass 0.001; collision sphere radius=0.01; visual sphere radius=0.01
- added link foot_contact_3, mass 0.001; collision sphere radius=0.01; visual sphere radius=0.01
- added link foot_contact_4, mass 0.001; collision sphere radius=0.01; visual sphere radius=0.01
- added link foot_contact_5, mass 0.001; collision sphere radius=0.01; visual sphere radius=0.01
- added link foot_contact_6, mass 0.001; collision sphere radius=0.01; visual sphere radius=0.01
- added link world
- link ankle_link_1: geometry collision cylinder length=0.203 radius=0.038; visual mesh filename=package://hexapod_description/meshes/ankle_link_1.STL
- link ankle_link_2: geometry collision cylinder length=0.203 radius=0.038; visual mesh filename=package://hexapod_description/meshes/ankle_link_1.STL
- link ankle_link_3: geometry collision cylinder length=0.203 radius=0.038; visual mesh filename=package://hexapod_description/meshes/ankle_link_1.STL
- link ankle_link_4: geometry collision cylinder length=0.203 radius=0.038; visual mesh filename=package://hexapod_description/meshes/ankle_link_1.STL
- link ankle_link_5: geometry collision cylinder length=0.203 radius=0.038; visual mesh filename=package://hexapod_description/meshes/ankle_link_1.STL
- link ankle_link_6: geometry collision cylinder length=0.203 radius=0.038; visual mesh filename=package://hexapod_description/meshes/ankle_link_1.STL
- link base_link: geometry collision cylinder length=0.064 radius=0.11; visual mesh filename=package://hexapod_description/meshes/base_link.STL
- link end_effector_1: geometry collision box size=0.032 0.022 0.022; visual mesh filename=package://hexapod_description/meshes/end_effector_1.STL
- link end_effector_2: geometry collision box size=0.032 0.022 0.022; visual mesh filename=package://hexapod_description/meshes/end_effector_1.STL
- link end_effector_3: geometry collision box size=0.032 0.022 0.022; visual mesh filename=package://hexapod_description/meshes/end_effector_1.STL
- link end_effector_4: geometry collision box size=0.032 0.022 0.022; visual mesh filename=package://hexapod_description/meshes/end_effector_1.STL
- link end_effector_5: geometry collision box size=0.032 0.022 0.022; visual mesh filename=package://hexapod_description/meshes/end_effector_1.STL
- link end_effector_6: geometry collision box size=0.032 0.022 0.022; visual mesh filename=package://hexapod_description/meshes/end_effector_1.STL
- link foot_pointer_1: geometry collision box size=0.032 0.023 0.022; visual mesh filename=package://hexapod_description/meshes/foot_pointer_1.STL
- link foot_pointer_2: geometry collision box size=0.032 0.023 0.022; visual mesh filename=package://hexapod_description/meshes/foot_pointer_1.STL
- link foot_pointer_3: geometry collision box size=0.032 0.023 0.022; visual mesh filename=package://hexapod_description/meshes/foot_pointer_1.STL
- link foot_pointer_4: geometry collision box size=0.032 0.023 0.022; visual mesh filename=package://hexapod_description/meshes/foot_pointer_1.STL
- link foot_pointer_5: geometry collision box size=0.032 0.023 0.022; visual mesh filename=package://hexapod_description/meshes/foot_pointer_1.STL
- link foot_pointer_6: geometry collision box size=0.032 0.023 0.022; visual mesh filename=package://hexapod_description/meshes/foot_pointer_1.STL
- link hip_link_1: mass 0.111649772064324 -> 0.0882011859976947; geometry collision box size=0.126 0.061 0.077; visual mesh filename=package://hexapod_description/meshes/hip_link_1.STL
- link hip_link_2: geometry collision box size=0.126 0.061 0.077; visual mesh filename=package://hexapod_description/meshes/hip_link_1.STL
- link hip_link_3: mass 0.0882011859976946 -> 0.0882011859976947; geometry collision box size=0.126 0.061 0.077; visual mesh filename=package://hexapod_description/meshes/hip_link_1.STL
- link hip_link_4: geometry collision box size=0.126 0.061 0.077; visual mesh filename=package://hexapod_description/meshes/hip_link_1.STL
- link hip_link_5: geometry collision box size=0.126 0.061 0.077; visual mesh filename=package://hexapod_description/meshes/hip_link_1.STL
- link hip_link_6: mass 0.0882011859976949 -> 0.0882011859976947; geometry collision box size=0.126 0.061 0.077; visual mesh filename=package://hexapod_description/meshes/hip_link_1.STL
- link knee_link_1: geometry collision box size=0.134 0.129 0.080; visual mesh filename=package://hexapod_description/meshes/knee_link_1.STL
- link knee_link_2: geometry collision box size=0.134 0.129 0.080; visual mesh filename=package://hexapod_description/meshes/knee_link_1.STL
- link knee_link_3: geometry collision box size=0.134 0.129 0.080; visual mesh filename=package://hexapod_description/meshes/knee_link_1.STL
- link knee_link_4: geometry collision box size=0.134 0.129 0.080; visual mesh filename=package://hexapod_description/meshes/knee_link_1.STL
- link knee_link_5: geometry collision box size=0.134 0.129 0.080; visual mesh filename=package://hexapod_description/meshes/knee_link_1.STL
- link knee_link_6: geometry collision box size=0.134 0.129 0.080; visual mesh filename=package://hexapod_description/meshes/knee_link_1.STL
Joints:
- added joint foot_contact_joint_1: type fixed, parent end_effector_1, child foot_contact_1, origin xyz=-0.012 0.0015 0 rpy=0 0 0
- added joint foot_contact_joint_2: type fixed, parent end_effector_2, child foot_contact_2, origin xyz=-0.012 0.0015 0 rpy=0 0 0
- added joint foot_contact_joint_3: type fixed, parent end_effector_3, child foot_contact_3, origin xyz=-0.012 0.0015 0 rpy=0 0 0
- added joint foot_contact_joint_4: type fixed, parent end_effector_4, child foot_contact_4, origin xyz=-0.012 0.0015 0 rpy=0 0 0
- added joint foot_contact_joint_5: type fixed, parent end_effector_5, child foot_contact_5, origin xyz=-0.012 0.0015 0 rpy=0 0 0
- added joint foot_contact_joint_6: type fixed, parent end_effector_6, child foot_contact_6, origin xyz=-0.012 0.0015 0 rpy=0 0 0
- added joint world_to_base: type fixed, parent world, child base_link, origin xyz=0 0 0.3 rpy=0 0 0
- joint ankle_joint_1: limit lower=0 upper=0 effort=0 velocity=0 -> lower=-3.14 upper=3.14 effort=20.0 velocity=5.0
- joint ankle_joint_2: limit lower=0 upper=0 effort=0 velocity=0 -> lower=-3.14 upper=3.14 effort=20.0 velocity=5.0
- joint ankle_joint_3: limit lower=0 upper=0 effort=0 velocity=0 -> lower=-3.14 upper=3.14 effort=20.0 velocity=5.0
- joint ankle_joint_4: limit lower=0 upper=0 effort=0 velocity=0 -> lower=-3.14 upper=3.14 effort=20.0 velocity=5.0
- joint ankle_joint_5: limit lower=0 upper=0 effort=0 velocity=0 -> lower=-3.14 upper=3.14 effort=20.0 velocity=5.0
- joint ankle_joint_6: limit lower=0 upper=0 effort=0 velocity=0 -> lower=-3.14 upper=3.14 effort=20.0 velocity=5.0
- joint end_effector_joint_1: axis 0 0 0 -> (none)
- joint end_effector_joint_2: axis 0 0 0 -> (none)
- joint end_effector_joint_3: axis 0 0 0 -> (none)
- joint end_effector_joint_4: axis 0 0 0 -> (none)
- joint end_effector_joint_5: axis 0 0 0 -> (none)
- joint end_effector_joint_6: axis 0 0 0 -> (none)
- joint foot_pointer_joint_1: axis 0 0 0 -> (none)
- joint foot_pointer_joint_2: axis 0 0 0 -> (none)
- joint foot_pointer_joint_3: axis 0 0 0 -> (none)
- joint foot_pointer_joint_4: axis 0 0 0 -> (none)
- joint foot_pointer_joint_5: axis 0 0 0 -> (none)
- joint foot_pointer_joint_6: axis 0 0 0 -> (none)
- joint hip_joint_1: limit lower=0 upper=0 effort=0 velocity=0 -> lower=-1.57 upper=1.57 effort=20.0 velocity=5.0
- joint hip_joint_2: limit lower=0 upper=0 effort=0 velocity=0 -> lower=-1.57 upper=1.57 effort=20.0 velocity=5.0
- joint hip_joint_3: limit lower=0 upper=0 effort=0 velocity=0 -> lower=-1.57 upper=1.57 effort=20.0 velocity=5.0
- joint hip_joint_4: limit lower=0 upper=0 effort=0 velocity=0 -> lower=-1.57 upper=1.57 effort=20.0 velocity=5.0
- joint hip_joint_5: limit lower=0 upper=0 effort=0 velocity=0 -> lower=-1.57 upper=1.57 effort=20.0 velocity=5.0
- joint hip_joint_6: limit lower=0 upper=0 effort=0 velocity=0 -> lower=-1.57 upper=1.57 effort=20.0 velocity=5.0
- joint knee_joint_1: limit lower=0 upper=0 effort=0 velocity=0 -> lower=-3.14 upper=3.14 effort=20.0 velocity=5.0
- joint knee_joint_2: limit lower=0 upper=0 effort=0 velocity=0 -> lower=-3.14 upper=3.14 effort=20.0 velocity=5.0
- joint knee_joint_3: limit lower=0 upper=0 effort=0 velocity=0 -> lower=-3.14 upper=3.14 effort=20.0 velocity=5.0
- joint knee_joint_4: limit lower=0 upper=0 effort=0 velocity=0 -> lower=-3.14 upper=3.14 effort=20.0 velocity=5.0
- joint knee_joint_5: limit lower=0 upper=0 effort=0 velocity=0 -> lower=-3.14 upper=3.14 effort=20.0 velocity=5.0
- joint knee_joint_6: limit lower=0 upper=0 effort=0 velocity=0 -> lower=-3.14 upper=3.14 effort=20.0 velocity=5.0

File: src/hexapod_description/robot/visual/hexapod_params.xacro (robot description, xacro)
@@ -26,5 +26,5 @@
     <xacro:property name="end_effector_joint_y" value="-0.00094278"/>
     <!-- JOINT LIMITS (radians) -->
-    <xacro:property name="joint_effort" value="10.0"/>
+    <xacro:property name="joint_effort" value="20.0"/>
     <xacro:property name="joint_velocity" value="5.0"/>
     <!-- Hip joint limits -->
@@ -32,19 +32,19 @@
     <xacro:property name="hip_upper_limit" value="1.57"/>
     <!-- Knee joint limits -->
-    <xacro:property name="knee_lower_limit" value="-2.0"/>
-    <xacro:property name="knee_upper_limit" value="2.0"/>
+    <xacro:property name="knee_lower_limit" value="-3.14"/>
+    <xacro:property name="knee_upper_limit" value="3.14"/>
     <!-- Ankle joint limits -->
-    <xacro:property name="ankle_lower_limit" value="-1.57"/>
-    <xacro:property name="ankle_upper_limit" value="1.57"/>
+    <xacro:property name="ankle_lower_limit" value="-3.14"/>
+    <xacro:property name="ankle_upper_limit" value="3.14"/>
     <!-- JOINT DYNAMICS -->
-    <!-- Hip joint -->
-    <xacro:property name="hip_damping" value="0.1"/>
-    <xacro:property name="hip_friction" value="0.05"/>
-    <!-- Knee joint -->
-    <xacro:property name="knee_damping" value="0.1"/>
-    <xacro:property name="knee_friction" value="0.05"/>
-    <!-- Ankle joint -->
-    <xacro:property name="ankle_damping" value="0.1"/>
-    <xacro:property name="ankle_friction" value="0.05"/>
+    <!-- Hip joint - Updated for PID tuning -->
+    <xacro:property name="hip_damping" value="0.019728"/>
+    <xacro:property name="hip_friction" value="0.01"/>
+    <!-- Knee joint - Updated for PID tuning -->
+    <xacro:property name="knee_damping" value="0.1"/>  <!-- INCREASED to reduce oscillation -->
+    <xacro:property name="knee_friction" value="0.01"/>
+    <!-- Ankle joint - Updated for PID tuning -->
+    <xacro:property name="ankle_damping" value="0.019728"/>
+    <xacro:property name="ankle_friction" value="0.01"/>
 <!-- FOOT CONTACT PARAMETERS -->
     <xacro:property name="foot_contact_radius" value="0.01"/>

File: src/hexapod_description/robot/visual/hexapod_trajectory.xacro (robot description, xacro)
@@ -4,8 +4,11 @@
     <xacro:include filename="$(find hexapod_description)/robot/visual/hexapod_params.xacro" />
     <xacro:include filename="$(find hexapod_description)/robot/visual/robot_material.xacro" />
-    <xacro:include filename="$(find hexapod_description)/robot/visual/gazebo_full.xacro" />
-    <!-- WORLD LINK (for fixing robot in air during tuning) -->
+    <xacro:include filename="$(find hexapod_description)/robot/visual/gazebo_trajectory.xacro" />
+    <!-- Property to enable/disable mesh rendering (for debugging) -->
+    <xacro:property name="use_mesh" value="true" />
+    <!-- WORLD LINK - Required for mesh rendering in Gazebo -->
     <link name="world"/>
-    <!-- FIXED JOINT (world to base_link - for PID tuning) -->
+    <!-- FIXED JOINT - Enables mesh rendering, keeps robot suspended for testing -->
+    <!-- NOTE: For walking simulation, this should be removed and robot spawned on ground -->
     <joint name="world_to_base" type="fixed">
         <parent link="world"/>
@@ -246,5 +249,5 @@
         </joint>
     </xacro:macro>
-    <!-- INSTANTIATE 6 LEGS -->
+    <!-- INSTANTIATE 6 LEGS - Using correct hexagonal layout from hexapod.xacro -->
     <xacro:hexapod_leg leg_num="1"
                        hip_origin_xyz="-1.2616E-05 -0.095255 0"
