Commit message: 001

File: src/hexapod_description/robot/visual/hexapod.xacro (robot description, xacro)
@@ -26,7 +26,7 @@
         </visual>
         <collision>
-            <origin xyz="0 0 0" rpy="0 0 0" />
+            <origin xyz="0 0 0.002" rpy="0 0 0" />
             <geometry>
-                <mesh filename="package://hexapod_description/meshes/base_link.STL" />
+                <cylinder radius="0.11" length="0.064"/>
             </geometry>
         </collision>
@@ -55,7 +55,7 @@
             </visual>
             <collision>
-                <origin xyz="0 0 0" rpy="0 0 0" />
-                <geometry>
-                    <mesh filename="package://hexapod_description/meshes/hip_link_1.STL" />
+                <origin xyz="0.0445 -0.0013 -0.0015" rpy="0 0 0" />
+                <geometry>
+                    <box size="0.126 0.061 0.077"/>
                 </geometry>
             </collision>
@@ -92,7 +92,7 @@
             </visual>
             <collision>
-                <origin xyz="0 0 0" rpy="0 0 0" />
-                <geometry>
-                    <mesh filename="package://hexapod_description/meshes/knee_link_1.STL" />
+                <origin xyz="-0.0484 -0.0449 -0.0011" rpy="0 0 0" />
+                <geometry>
+                    <box size="0.134 0.129 0.080"/>
                 </geometry>
             </collision>
@@ -130,7 +130,7 @@
             </visual>
             <collision>
-                <origin xyz="0 0 0" rpy="0 0 0" />
-                <geometry>
-                    <mesh filename="package://hexapod_description/meshes/ankle_link_1.STL" />
+                <origin xyz="0.0717 -0.0069 -0.0059" rpy="0 1.5708 0" />
+                <geometry>
+                    <cylinder radius="0.038" length="0.203"/>
                 </geometry>
             </collision>
@@ -167,7 +167,7 @@
             </visual>
             <collision>
-                <origin xyz="0 0 0" rpy="0 0 0" />
-                <geometry>
-                    <mesh filename="package://hexapod_description/meshes/foot_pointer_1.STL" />
+                <origin xyz="-0.0081 0.0008 0" rpy="0 0 0" />
+                <geometry>
+                    <box size="0.032 0.023 0.022"/>
                 </geometry>
             </collision>
@@ -200,7 +200,7 @@
             </visual>
             <collision>
-                <origin xyz="0 0 0" rpy="0 0 0" />
-                <geometry>
-                    <mesh filename="package://hexapod_description/meshes/end_effector_1.STL" />
+                <origin xyz="-0.0157 0.0014 0" rpy="0 0 0" />
+                <geometry>
+                    <box size="0.032 0.022 0.022"/>
                 </geometry>
             </collision>
@@ -212,5 +212,5 @@
             <child link="end_effector_${leg_num}" />
         </joint>
-        <!-- FOOT CONTACT SPHERE (for simulation/collision) -->
+        <!-- FOOT CONTACT SPHERE -->
         <link name="foot_contact_${leg_num}">
             <xacro:inertial_sphere mass="${foot_contact_mass}" radius="${foot_contact_radius}">
@@ -239,25 +239,19 @@
     </xacro:macro>
     <!-- INSTANTIATE 6 LEGS -->
-    <!-- Leg 1: Rear Right -->
     <xacro:hexapod_leg leg_num="1"
                        hip_origin_xyz="-1.2616E-05 -0.095255 0"
                        hip_origin_rpy="0 0 -1.5708" />
-    <!-- Leg 2: Front Right -->
     <xacro:hexapod_leg leg_num="2"
                        hip_origin_xyz="0.082487 -0.047638 0"
                        hip_origin_rpy="0 0 -0.5236" />
-    <!-- Leg 3: Front Left -->
     <xacro:hexapod_leg leg_num="3"
                        hip_origin_xyz="0.082499 0.047616 0"
                        hip_origin_rpy="0 0 0.5236" />
-    <!-- Leg 4: Rear Left -->
     <xacro:hexapod_leg leg_num="4"
                        hip_origin_xyz="1.2616E-05 0.095255 0"
                        hip_origin_rpy="0 0 1.5708" />
-    <!-- Leg 5: Middle Left -->
     <xacro:hexapod_leg leg_num="5"
                        hip_origin_xyz="-0.082487 0.047638 0"
                        hip_origin_rpy="0 0 2.618" />
-    <!-- Leg 6: Middle Right -->
     <xacro:hexapod_leg leg_num="6"
                        hip_origin_xyz="-0.082499 -0.047616 0"

Commit message: add platform and change trajectory into  something more simple

File: src/hexapod_description/robot/visual/hexapod.xacro (robot description, xacro)
@@ -5,4 +5,9 @@
     <xacro:include filename="$(find hexapod_description)/robot/visual/robot_material.xacro" />
     <xacro:include filename="$(find hexapod_description)/robot/visual/gazebo_full.xacro" />
+    <xacro:include filename="$(find hexapod_description)/robot/visual/cylinder_platform.xacro" />
+    <!-- CYLINDRICAL PLATFORM -->
+    <xacro:cylinder_platform name="base_platform" parent="base_link" radius="0.15" height="1.0">
+        <origin xyz="0 0 -0.5" rpy="0 0 0"/>
+    </xacro:cylinder_platform>
     <!-- BASE LINK -->
     <link name="base_link">
