Commit message: update

File: src/hexapod_description/robot/visual/gazebo_full.xacro (robot description, xacro)
@@ -1,6 +1,5 @@
 <?xml version="1.0"?>
-<robot xmlns:xacro="http://www.ros.org/wiki/xacro">
-  <!-- ros2_control for Gazebo Sim (Ignition) -->
-  <ros2_control name="HexapodGazeboSystem" type="system">
+<robot xmlns:xacro="http://www.ros.org/wiki/xacro" name="hexapod">
+  <ros2_control name="GazeboSimSystem" type="system">
     <hardware>
       <plugin>gz_ros2_control/GazeboSimSystem</plugin>
@@ -9,6 +8,6 @@
     <joint name="hip_joint_1">
       <command_interface name="effort">
-        <param name="min">-10</param>
-        <param name="max">10</param>
+        <param name="min">-100</param>
+        <param name="max">100</param>
       </command_interface>
       <state_interface name="position">
@@ -20,6 +19,6 @@
     <joint name="knee_joint_1">
       <command_interface name="effort">
-        <param name="min">-10</param>
-        <param name="max">10</param>
+        <param name="min">-100</param>
+        <param name="max">100</param>
       </command_interface>
       <state_interface name="position">
@@ -31,6 +30,6 @@
     <joint name="ankle_joint_1">
       <command_interface name="effort">
-        <param name="min">-10</param>
-        <param name="max">10</param>
+        <param name="min">-100</param>
+        <param name="max">100</param>
       </command_interface>
       <state_interface name="position">
@@ -43,6 +42,6 @@
     <joint name="hip_joint_2">
       <command_interface name="effort">
-        <param name="min">-10</param>
-        <param name="max">10</param>
+        <param name="min">-100</param>
+        <param name="max">100</param>
       </command_interface>
       <state_interface name="position">
@@ -54,6 +53,6 @@
     <joint name="knee_joint_2">
       <command_interface name="effort">
-        <param name="min">-10</param>
-        <param name="max">10</param>
+        <param name="min">-100</param>
+        <param name="max">100</param>
       </command_interface>
       <state_interface name="position">
@@ -65,6 +64,6 @@
     <joint name="ankle_joint_2">
       <command_interface name="effort">
-        <param name="min">-10</param>
-        <param name="max">10</param>
+        <param name="min">-100</param>
+        <param name="max">100</param>
       </command_interface>
       <state_interface name="position">
@@ -77,6 +76,6 @@
     <joint name="hip_joint_3">
       <command_interface name="effort">
-        <param name="min">-10</param>
-        <param name="max">10</param>
+        <param name="min">-100</param>
+        <param name="max">100</param>
       </command_interface>
       <state_interface name="position">
@@ -88,6 +87,6 @@
     <joint name="knee_joint_3">
       <command_interface name="effort">
-        <param name="min">-10</param>
-        <param name="max">10</param>
+        <param name="min">-100</param>
+        <param name="max">100</param>
       </command_interface>
       <state_interface name="position">
@@ -99,6 +98,6 @@
     <joint name="ankle_joint_3">
       <command_interface name="effort">
-        <param name="min">-10</param>
-        <param name="max">10</param>
+        <param name="min">-100</param>
+        <param name="max">100</param>
       </command_interface>
       <state_interface name="position">
@@ -111,6 +110,6 @@
     <joint name="hip_joint_4">
       <command_interface name="effort">
-        <param name="min">-10</param>
-        <param name="max">10</param>
+        <param name="min">-100</param>
+        <param name="max">100</param>
       </command_interface>
       <state_interface name="position">
@@ -122,6 +121,6 @@
     <joint name="knee_joint_4">
       <command_interface name="effort">
-        <param name="min">-10</param>
-        <param name="max">10</param>
+        <param name="min">-100</param>
+        <param name="max">100</param>
       </command_interface>
       <state_interface name="position">
@@ -133,6 +132,6 @@
     <joint name="ankle_joint_4">
       <command_interface name="effort">
-        <param name="min">-10</param>
-        <param name="max">10</param>
+        <param name="min">-100</param>
+        <param name="max">100</param>
       </command_interface>
       <state_interface name="position">
@@ -145,6 +144,6 @@
     <joint name="hip_joint_5">
       <command_interface name="effort">
-        <param name="min">-10</param>
-        <param name="max">10</param>
+        <param name="min">-100</param>
+        <param name="max">100</param>
       </command_interface>
       <state_interface name="position">
@@ -156,6 +155,6 @@
     <joint name="knee_joint_5">
       <command_interface name="effort">
-        <param name="min">-10</param>
-        <param name="max">10</param>
+        <param name="min">-100</param>
+        <param name="max">100</param>
       </command_interface>
       <state_interface name="position">
@@ -167,6 +166,6 @@
     <joint name="ankle_joint_5">
       <command_interface name="effort">
-        <param name="min">-10</param>
-        <param name="max">10</param>
+        <param name="min">-100</param>
+        <param name="max">100</param>
       </command_interface>
       <state_interface name="position">
@@ -179,6 +178,6 @@
     <joint name="hip_joint_6">
       <command_interface name="effort">
-        <param name="min">-10</param>
-        <param name="max">10</param>
+        <param name="min">-100</param>
+        <param name="max">100</param>
       </command_interface>
       <state_interface name="position">
@@ -190,6 +189,6 @@
     <joint name="knee_joint_6">
       <command_interface name="effort">
-        <param name="min">-10</param>
-        <param name="max">10</param>
+        <param name="min">-100</param>
+        <param name="max">100</param>
       </command_interface>
       <state_interface name="position">
@@ -201,6 +200,6 @@
     <joint name="ankle_joint_6">
       <command_interface name="effort">
-        <param name="min">-10</param>
-        <param name="max">10</param>
+        <param name="min">-100</param>
+        <param name="max">100</param>
       </command_interface>
       <state_interface name="position">
@@ -211,45 +210,26 @@
     </joint>
   </ros2_control>
-  <!-- Gazebo ros2_control Plugin -->
   <gazebo>
     <plugin filename="gz_ros2_control-system" name="gz_ros2_control::GazeboSimROS2ControlPlugin">
       <parameters>$(find hexapod_simulation)/config/controller_full.yaml</parameters>
     </plugin>
+    <!-- Sensor Manager (for IMU, Lidar, etc.) -->
+    <plugin filename="libignition-gazebo-sensors-system.so"
+            name="ignition::gazebo::systems::Sensors">
+      <render_engine>ogre2</render_engine>
+    </plugin>
   </gazebo>
-  <!-- Ground Contact Plugin for all foot contacts -->
-  <xacro:macro name="foot_contact_sensor" params="leg_num">
-    <gazebo reference="foot_contact_${leg_num}">
-      <sensor name="foot_contact_sensor_${leg_num}" type="contact">
-        <contact>
-          <collision>foot_contact_${leg_num}_collision</collision>
-        </contact>
-        <always_on>true</always_on>
-        <update_rate>100</update_rate>
-      </sensor>
-      <!-- Contact surface properties -->
-      <mu1>0.8</mu1>
-      <mu2>0.8</mu2>
-      <kp>1000000.0</kp>
-      <kd>100.0</kd>
-      <minDepth>0.001</minDepth>
-      <maxVel>0.01</maxVel>
-    </gazebo>
-  </xacro:macro>
-  <!-- Instantiate contact sensors for all 6 legs -->
-  <xacro:foot_contact_sensor leg_num="1"/>
-  <xacro:foot_contact_sensor leg_num="2"/>
-  <xacro:foot_contact_sensor leg_num="3"/>
-  <xacro:foot_contact_sensor leg_num="4"/>
-  <xacro:foot_contact_sensor leg_num="5"/>
-  <xacro:foot_contact_sensor leg_num="6"/>
-  <!-- IMU Sensor on Base Link -->
-  <gazebo reference="base_link">
+  <!-- Optional IMU sensor on base_link -->
+  <!-- <gazebo reference="base_link">
     <sensor name="imu_sensor" type="imu">
       <always_on>true</always_on>
-      <update_rate>100</update_rate>
+      <update_rate>100.0</update_rate>
       <visualize>true</visualize>
-      <topic>imu_data</topic>
-      <enable_metrics>false</enable_metrics>
+      <topic>/imu/data</topic>
+      <gz_frame_id>base_link</gz_frame_id>
+      <plugin filename="libignition-gazebo-imu-system.so"
+              name="ignition::gazebo::systems::Imu"/>
+      <pose>0 0 0 0 0 0</pose>
     </sensor>
-  </gazebo>
+  </gazebo> -->
 </robot>

Commit message: fucking hopeless progress

File: src/hexapod_description/robot/visual/gazebo_full.xacro (robot description, xacro)
@@ -218,4 +218,13 @@
             name="ignition::gazebo::systems::Sensors">
       <render_engine>ogre2</render_engine>
+    </plugin>
+    <!-- Pose Publisher: Publishes world->base_link transform to TF -->
+    <!-- This ensures Gazebo's world frame matches RViz's world frame -->
+    <plugin filename="libignition-gazebo-pose-publisher-system.so"
+            name="ignition::gazebo::systems::PosePublisher">
+      <publish_link_pose>true</publish_link_pose>
+      <use_pose_vector_msg>false</use_pose_vector_msg>
+      <static_publisher>false</static_publisher>
+      <static_update_frequency>100.0</static_update_frequency>
     </plugin>
   </gazebo>

File: src/hexapod_description/robot/visual/hexapod.xacro (robot description, xacro)
@@ -5,4 +5,17 @@
     <xacro:include filename="$(find hexapod_description)/robot/visual/robot_material.xacro" />
     <xacro:include filename="$(find hexapod_description)/robot/visual/gazebo_full.xacro" />
+    <!-- WORLD FRAME -->
+    <!-- This is the fixed reference frame for both Gazebo and RViz -->
+    <link name="world"/>
+    <!-- WORLD TO BASE_LINK JOINT -->
+    <!-- This joint defines the position of the hexapod relative to the world frame -->
+    <!-- In Gazebo, this will be automatically handled by physics, but we define it here -->
+    <!-- for proper TF tree structure in RViz -->
+    <joint name="world_to_base" type="fixed">
+        <parent link="world"/>
+        <child link="base_link"/>
+        <!-- Robot frame is 2m below world frame (world is 2m above robot) -->
+        <origin xyz="5.0 0.0 0.0" rpy="0 0 0"/>
+    </joint>
     <!-- BASE LINK -->
     <link name="base_link">

Commit message: Change Kinematic System

File: src/hexapod_description/robot/visual/gazebo_full.xacro (robot description, xacro)
@@ -218,13 +218,4 @@
             name="ignition::gazebo::systems::Sensors">
       <render_engine>ogre2</render_engine>
-    </plugin>
-    <!-- Pose Publisher: Publishes world->base_link transform to TF -->
-    <!-- This ensures Gazebo's world frame matches RViz's world frame -->
-    <plugin filename="libignition-gazebo-pose-publisher-system.so"
-            name="ignition::gazebo::systems::PosePublisher">
-      <publish_link_pose>true</publish_link_pose>
-      <use_pose_vector_msg>false</use_pose_vector_msg>
-      <static_publisher>false</static_publisher>
-      <static_update_frequency>100.0</static_update_frequency>
     </plugin>
   </gazebo>

File: src/hexapod_description/robot/visual/hexapod.xacro (robot description, xacro)
@@ -5,17 +5,4 @@
     <xacro:include filename="$(find hexapod_description)/robot/visual/robot_material.xacro" />
     <xacro:include filename="$(find hexapod_description)/robot/visual/gazebo_full.xacro" />
-    <!-- WORLD FRAME -->
-    <!-- This is the fixed reference frame for both Gazebo and RViz -->
-    <link name="world"/>
-    <!-- WORLD TO BASE_LINK JOINT -->
-    <!-- This joint defines the position of the hexapod relative to the world frame -->
-    <!-- In Gazebo, this will be automatically handled by physics, but we define it here -->
-    <!-- for proper TF tree structure in RViz -->
-    <joint name="world_to_base" type="fixed">
-        <parent link="world"/>
-        <child link="base_link"/>
-        <!-- Robot frame is 2m below world frame (world is 2m above robot) -->
-        <origin xyz="5.0 0.0 0.0" rpy="0 0 0"/>
-    </joint>
     <!-- BASE LINK -->
     <link name="base_link">
